Commit message: lame example working

File: 7DofArm.urdf (robot description, URDF)
Before this commit: robot robot_name, 9 links, 8 joints
Links:
- link link_1: geometry visual cylinder length=.15 radius=0.075; visual cylinder length=1 radius=0.05
- link link_2: geometry visual cylinder length=.15 radius=0.075; visual cylinder length=1 radius=0.05
- link link_3: geometry visual cylinder length=.15 radius=0.075; visual cylinder length=1 radius=0.05
- link link_4: geometry visual cylinder length=.15 radius=0.075; visual cylinder length=1 radius=0.05
- link link_5: geometry visual cylinder length=.15 radius=0.075; visual cylinder length=1 radius=0.05
- link link_6: geometry visual cylinder length=.15 radius=0.075; visual cylinder length=1 radius=0.05
- link link_7: geometry visual cylinder length=.15 radius=0.075; visual cylinder length=1 radius=0.05
- link tool: geometry visual sphere radius=.075
Joints:
- joint joint_1: limit lower=-6 upper=6 effort=1000.0 velocity=1.57 -> (none)
- joint joint_2: limit lower=-6 upper=6 effort=1000.0 velocity=0.5 -> (none)
- joint joint_3: limit lower=-6 upper=6 effort=1000.0 velocity=0.5 -> (none)
- joint joint_4: limit lower=-6 upper=6 effort=1000.0 velocity=0.5 -> (none)
- joint joint_5: limit lower=-6 upper=6 effort=1000.0 velocity=0.5 -> (none)
- joint joint_6: limit lower=-6 upper=6 effort=1000.0 velocity=0.5 -> (none)
- joint joint_7: limit lower=-6 upper=6 effort=1000.0 velocity=0.5 -> (none)
